File: tps61165_led_driver.sch (KiCad schematic (older format))
At the start: 12 parts, among them K1 CONN_3, P1 CONN_2, U1 TPS61165_DBV_6_DBV6

Commit message: ADD: pdf
Parts:
- added P2, P3: CONN_1, symbol CONN_1
Connections:
- net Vin: now reaches C1.1, C2.1, K1.2 (PM), L1.2, U1.1 (VIN)
- net Ctrl: now reaches K1.3 (P3), U1.2 (CTRL)
- net GND: now reaches C1.2, C2.2, C3.2, C4.2, C5.2, K1.1 (P1), R2.2, U1.4 (GND)
- net GND: now also R1.2
- net Comp: now reaches C3.1, U1.5 (COMP)
- net FB: now reaches P1.1 (P1), R1.1, U1.6 (FB)
- net FB: now also R2.1
Other:
- moved on the sheet: R2
Changed lines of the file:
@@
 LIBS:SparkFun
 LIBS:SparkFun-Connectors
-EELAYER 27 0
+LIBS:tps61165_led_driver-cache
+EELAYER 24 0
 EELAYER END
 $Descr A4 11693 8268
@@
 U 1 1 550EFBF6
 P 5200 4400
-F 0 "U1" H 5200 4400 0   0001 C CNN
-F 1 "TPS61165_DBV_6_DBV6" H 5200 4400 0   0001 C CNN
+F 0 "U1" H 5200 4400 60  0001 C CNN
+F 1 "TPS61165_DBV_6_DBV6" H 5200 4400 60  0001 C CNN
 F 2 "" H 5200 4400 60  0000 C CNN
 F 3 "" H 5200 4400 60  0000 C CNN
@@
 L R R2
 U 1 1 550EFD3A
-P 6350 5050
-F 0 "R2" V 6430 5050 40  0000 C CNN
-F 1 "R" V 6357 5051 40  0000 C CNN
-F 2 "~" V 6280 5050 30  0000 C CNN
-F 3 "~" H 6350 5050 30  0000 C CNN
-	1    6350 5050
-	1    0    0    -1
-$EndComp
-Wire Wire Line
-	6350 5550 6350 5300
+P 6500 4550
+F 0 "R2" V 6580 4550 40  0000 C CNN
+F 1 "R" V 6507 4551 40  0000 C CNN
+F 2 "~" V 6430 4550 30  0000 C CNN
+F 3 "~" H 6500 4550 30  0000 C CNN
+	1    6500 4550
+	1    0    0    -1
+$EndComp
+Wire Wire Line
+	6350 4800 6350 5550
 Connection ~ 6350 5550
 Wire Wire Line
-	6350 4300 5800 4300
+	5800 4300 6500 4300
 Wire Wire Line
 	7400 4100 6350 4100
@@
 Wire Wire Line
 	4200 5100 4400 5100
+Wire Wire Line
+	6500 4800 6500 5550
+Connection ~ 6500 5550
+Text Label 3400 4150 0    60   ~ 0
+Ctrl
+Text Label 3400 4250 0    60   ~ 0
+Vin
+Text Label 3400 4350 0    60   ~ 0
+GND
+Text Label 6000 4400 0    60   ~ 0
+Comp
+Text Label 6350 4300 0    60   ~ 0
+FB
+$Comp
+L CONN_1 P2
+U 1 1 55101E32
+P 5300 3000
+F 0 "P2" H 5380 3000 40  0000 L CNN
+F 1 "CONN_1" H 5300 3055 30  0001 C CNN
+F 2 "" H 5300 3000 60  0000 C CNN
+F 3 "" H 5300 3000 60  0000 C CNN
+	1    5300 3000
+	1    0    0    -1
+$EndComp
+$Comp
+L CONN_1 P3
+U 1 1 55101E3F
+P 5300 3150
+F 0 "P3" H 5380 3150 40  0000 L CNN
+F 1 "CONN_1" H 5300 3205 30  0001 C CNN
+F 2 "" H 5300 3150 60  0000 C CNN
+F 3 "" H 5300 3150 60  0000 C CNN
+	1    5300 3150
+	1    0    0    -1
+$EndComp
 $EndSCHEMATC

Commit message: ADD: pdf, added cap
Parts:
- added C6: C, ~, symbol C
Connections:
- net Comp: now also C6.1
- net GND: now also C6.2
Changed lines of the file:
@@
 Connection ~ 5800 5550
 Wire Wire Line
-	5800 4400 6000 4400
+	5800 4400 6150 4400
 Wire Wire Line
 	6000 4800 6000 5550
@@
 	1    0    0    -1
 $EndComp
+$Comp
+L C C6
+U 1 1 551068A3
+P 6150 4600
+F 0 "C6" H 6150 4700 40  0000 L CNN
+F 1 "C" H 6156 4515 40  0000 L CNN
+F 2 "~" H 6188 4450 30  0000 C CNN
+F 3 "~" H 6150 4600 60  0000 C CNN
+	1    6150 4600
+	1    0    0    -1
+$EndComp
+Wire Wire Line
+	6150 4800 6150 5550
+Connection ~ 6150 5550
+Connection ~ 6000 4400
 $EndSCHEMATC
